File: Hardware/HiBeam_8-pack_v02.sch (KiCad schematic (older format))
At the start: 24 parts, among them J1 CI, J2 DI, J3 5V, J4 GND, J5 CO, J6 DO, J7 5V, J8 GND, U1 APA102, U2 APA102, U3 APA102, U4 APA102, U5 APA102, U6 APA102, U7 APA102, U8 APA102

Commit message: Added gerbers, .gitignore and .gitattributes.
Parts:
- added LOGO?: SFE_LOGO_FLAME1_INCH, SFE_LOGO_FLAME_.9, symbol SFE_LOGO_FLAME1_INCH
- added LOGO?: OSHW-LOGOMINI, OSHW-LOGO-MINI, symbol OSHW-LOGOMINI
Changed lines of the file:
@@
 LIBS:SparkFun-RF
 LIBS:SparkFun-Sensors
-LIBS:HiBeam 8-pack v02-cache
+LIBS:HiBeam_8-pack_v02-cache
 EELAYER 26 0
 EELAYER END
@@
 	2000 4850 2150 4850
 Connection ~ 2150 5300
+$Comp
+L SFE_LOGO_FLAME1_INCH LOGO?
+U 1 1 591CA394
+P 6350 7600
+F 0 "LOGO?" H 6350 7600 50  0001 C CNN
+F 1 "SFE_LOGO_FLAME1_INCH" H 6350 7600 50  0001 C CNN
+F 2 "SFE_LOGO_FLAME_.9" H 6380 7750 20  0001 C CNN
+F 3 "" H 6350 7600 60  0001 C CNN
+	1    6350 7600
+	1    0    0    -1
+$EndComp
+$Comp
+L OSHW-LOGOMINI LOGO?
+U 1 1 591CA41A
+P 5700 7250
+F 0 "LOGO?" H 5700 7250 50  0001 C CNN
+F 1 "OSHW-LOGOMINI" H 5700 7250 50  0001 C CNN
+F 2 "OSHW-LOGO-MINI" H 5730 7400 20  0001 C CNN
+F 3 "" H 5700 7250 60  0001 C CNN
+	1    5700 7250
+	1    0    0    -1
+$EndComp
 $EndSCHEMATC

Commit message: Fixes after double check.
Parts:
- removed LOGO?: SFE_LOGO_FLAME1_INCH, SFE_LOGO_FLAME_.9, symbol SFE_LOGO_FLAME1_INCH
- added LOGO?: SFE_LOGO_NAME_FLAME.1_INCH, SFE_LOGO_NAME_FLAME_.1, symbol SFE_LOGO_NAME_FLAME.1_INCH
- C1, C2, C3, C4, C5, C6, C7, C8: value C -> 0.1uF
Other:
- note added: "1"
- note added: "Designed by Pete Dokter"
- note added: "Released under the Creative Commons\nAttribution Share-Alike 4.0 License\nhttps://creativecommons.org/licenses/by-sa/4.0/"
Changed lines of the file:
@@
 P 3900 2100
 F 0 "C1" V 3850 2000 50  0000 C CNN
-F 1 "C" V 3850 2200 50  0000 C CNN
+F 1 "0.1uF" V 3850 2250 50  0000 C CNN
 F 2 "SparkFun-Capacitors:0603" H 3938 1950 50  0001 C CNN
 F 3 "" H 3900 2100 50  0001 C CNN
@@
 P 5300 2100
 F 0 "C2" V 5250 2000 50  0000 C CNN
-F 1 "C" V 5250 2200 50  0000 C CNN
+F 1 "0.1uF" V 5250 2250 50  0000 C CNN
 F 2 "SparkFun-Capacitors:0603" H 5338 1950 50  0001 C CNN
 F 3 "" H 5300 2100 50  0001 C CNN
@@
 P 6700 2100
 F 0 "C3" V 6650 2000 50  0000 C CNN
-F 1 "C" V 6650 2200 50  0000 C CNN
+F 1 "0.1uF" V 6650 2250 50  0000 C CNN
 F 2 "SparkFun-Capacitors:0603" H 6738 1950 50  0001 C CNN
 F 3 "" H 6700 2100 50  0001 C CNN
@@
 P 8100 2100
 F 0 "C4" V 8050 2000 50  0000 C CNN
-F 1 "C" V 8050 2200 50  0000 C CNN
+F 1 "0.1uF" V 8050 2250 50  0000 C CNN
 F 2 "SparkFun-Capacitors:0603" H 8138 1950 50  0001 C CNN
 F 3 "" H 8100 2100 50  0001 C CNN
@@
 P 3900 3800
 F 0 "C5" V 3850 3700 50  0000 C CNN
-F 1 "C" V 3850 3900 50  0000 C CNN
+F 1 "0.1uF" V 3850 3900 50  0000 C CNN
 F 2 "SparkFun-Capacitors:0603" H 3938 3650 50  0001 C CNN
 F 3 "" H 3900 3800 50  0001 C CNN
@@
 P 5300 3800
 F 0 "C6" V 5250 3700 50  0000 C CNN
-F 1 "C" V 5250 3900 50  0000 C CNN
+F 1 "0.1uF" V 5250 3950 50  0000 C CNN
 F 2 "SparkFun-Capacitors:0603" H 5338 3650 50  0001 C CNN
 F 3 "" H 5300 3800 50  0001 C CNN
@@
 P 6700 3800
 F 0 "C7" V 6650 3700 50  0000 C CNN
-F 1 "C" V 6650 3900 50  0000 C CNN
+F 1 "0.1uF" V 6650 3950 50  0000 C CNN
 F 2 "SparkFun-Capacitors:0603" H 6738 3650 50  0001 C CNN
 F 3 "" H 6700 3800 50  0001 C CNN
@@
 P 8100 3800
 F 0 "C8" V 8050 3700 50  0000 C CNN
-F 1 "C" V 8050 3900 50  0000 C CNN
+F 1 "0.1uF" V 8050 3950 50  0000 C CNN
 F 2 "SparkFun-Capacitors:0603" H 8138 3650 50  0001 C CNN
 F 3 "" H 8100 3800 50  0001 C CNN
@@
 U 1 1 59135F76
 P 1700 3700
-F 0 "J3" H 1500 3750 50  0000 C CNN
-F 1 "5V" H 1500 3650 50  0000 C CNN
+F 0 "J3" H 1700 3850 50  0000 C CNN
+F 1 "5V" H 1700 3550 50  0000 C CNN
 F 2 "Pete:solder_pad_2" H 1730 3850 20  0001 C CNN
 F 3 "" H 1700 3700 60  0000 C CNN
@@
 U 1 1 5913608D
 P 1700 5300
-F 0 "J4" H 1500 5350 50  0000 C CNN
-F 1 "GND" H 1500 5250 50  0000 C CNN
+F 0 "J4" H 1700 5450 50  0000 C CNN
+F 1 "GND" H 1700 5150 50  0000 C CNN
 F 2 "Pete:solder_pad_2" H 1730 5450 20  0001 C CNN
 F 3 "" H 1700 5300 60  0000 C CNN
@@
 U 1 1 59136101
 P 1700 2200
-F 0 "J1" H 1500 2250 50  0000 C CNN
-F 1 "CI" H 1500 2150 50  0000 C CNN
+F 0 "J1" H 1700 2350 50  0000 C CNN
+F 1 "CI" H 1700 2050 50  0000 C CNN
 F 2 "Pete:solder_pad_2" H 1730 2350 20  0001 C CNN
 F 3 "" H 1700 2200 60  0000 C CNN
@@
 U 1 1 5913616A
 P 1700 2900
-F 0 "J2" H 1500 2950 50  0000 C CNN
-F 1 "DI" H 1500 2850 50  0000 C CNN
+F 0 "J2" H 1700 3050 50  0000 C CNN
+F 1 "DI" H 1700 2750 50  0000 C CNN
 F 2 "Pete:solder_pad_2" H 1730 3050 20  0001 C CNN
 F 3 "" H 1700 2900 60  0000 C CNN
@@
 U 1 1 591361D8
 P 9650 3900
-F 0 "J5" H 9500 3850 50  0000 R CNN
-F 1 "CO" H 9500 3950 50  0000 R CNN
+F 0 "J5" H 9700 3750 50  0000 R CNN
+F 1 "CO" H 9700 4050 50  0000 R CNN
 F 2 "Pete:solder_pad_2" H 9680 4050 20  0001 C CNN
 F 3 "" H 9650 3900 60  0000 C CNN
@@
 U 1 1 591362B3
 P 9650 4600
-F 0 "J6" H 9500 4550 50  0000 R CNN
-F 1 "DO" H 9500 4650 50  0000 R CNN
+F 0 "J6" H 9700 4450 50  0000 R CNN
+F 1 "DO" H 9700 4750 50  0000 R CNN
 F 2 "Pete:solder_pad_2" H 9680 4750 20  0001 C CNN
 F 3 "" H 9650 4600 60  0000 C CNN
@@
 	1    0    0    -1
 $EndComp
-Text Notes 10600 7650 0    60   ~ 12
+Text Notes 10600 7650 0    60   ~ 0
 v02
-Text Notes 8250 7650 0    60   ~ 12
+Text Notes 8250 7650 0    60   ~ 0
 5/15/17
-Text Notes 7350 7500 0    60   ~ 12
+Text Notes 7350 7500 0    60   ~ 0
 HiBeam 8-pack
 $Comp
@@
 U 1 1 591A7CA4
 P 1700 4150
-F 0 "J7" H 1500 4200 50  0000 C CNN
-F 1 "5V" H 1500 4100 50  0000 C CNN
+F 0 "J7" H 1700 4300 50  0000 C CNN
+F 1 "5V" H 1700 4000 50  0000 C CNN
 F 2 "Pete:solder_pad_2" H 1730 4300 20  0001 C CNN
 F 3 "" H 1700 4150 60  0000 C CNN
@@
 U 1 1 591A7E0C
 P 1700 4850
-F 0 "J8" H 1500 4900 50  0000 C CNN
-F 1 "GND" H 1500 4800 50  0000 C CNN
+F 0 "J8" H 1700 5000 50  0000 C CNN
+F 1 "GND" H 1700 4700 50  0000 C CNN
 F 2 "Pete:solder_pad_2" H 1730 5000 20  0001 C CNN
 F 3 "" H 1700 4850 60  0000 C CNN
@@
 Connection ~ 2150 5300
 $Comp
-L SFE_LOGO_FLAME1_INCH LOGO?
-U 1 1 591CA394
-P 6350 7600
-F 0 "LOGO?" H 6350 7600 50  0001 C CNN
-F 1 "SFE_LOGO_FLAME1_INCH" H 6350 7600 50  0001 C CNN
-F 2 "SFE_LOGO_FLAME_.9" H 6380 7750 20  0001 C CNN
-F 3 "" H 6350 7600 60  0001 C CNN
-	1    6350 7600
-	1    0    0    -1
-$EndComp
-$Comp
 L OSHW-LOGOMINI LOGO?
 U 1 1 591CA41A
-P 5700 7250
-F 0 "LOGO?" H 5700 7250 50  0001 C CNN
-F 1 "OSHW-LOGOMINI" H 5700 7250 50  0001 C CNN
-F 2 "OSHW-LOGO-MINI" H 5730 7400 20  0001 C CNN
-F 3 "" H 5700 7250 60  0001 C CNN
-	1    5700 7250
-	1    0    0    -1
-$EndComp
+P 6250 7250
+F 0 "LOGO?" H 6250 7250 50  0001 C CNN
+F 1 "OSHW-LOGOMINI" H 6250 7250 50  0001 C CNN
+F 2 "OSHW-LOGO-MINI" H 6280 7400 20  0001 C CNN
+F 3 "" H 6250 7250 60  0001 C CNN
+	1    6250 7250
+	1    0    0    -1
+$EndComp
+Text Notes 7020 6941 0    79   ~ 0
+Released under the Creative Commons\nAttribution Share-Alike 4.0 License\nhttps://creativecommons.org/licenses/by-sa/4.0/
+Text Notes 7280 7247 0    60   ~ 0
+1
+Text Notes 7388 7244 0    60   ~ 0
+1
+Text Notes 7026 7085 0    79   ~ 0
+Designed by Pete Dokter
+$Comp
+L SFE_LOGO_NAME_FLAME.1_INCH LOGO?
+U 1 1 591F53CA
+P 3400 7750
+F 0 "LOGO?" H 3400 7750 50  0001 C CNN
+F 1 "SFE_LOGO_NAME_FLAME.1_INCH" H 3400 7750 50  0001 C CNN
+F 2 "SFE_LOGO_NAME_FLAME_.1" H 3430 7900 20  0001 C CNN
+F 3 "" H 3400 7750 60  0001 C CNN
+	1    3400 7750
+	1    0    0    -1
+$EndComp
