File: Hardware/HiBeam_8-pack_v02.kicad_pcb (KiCad board)
At the start: 2 copper layers, 28.4 x 28.4 mm, 38 parts, among them J1 M01PTH, J2 M01PTH, J3 M01PTH, J4 M01PTH, J5 M01PTH, J6 M01PTH, J7 M01PTH, J8 M01PTH, U1 APA102, U2 APA102, U3 APA102, U4 APA102, U5 APA102, U6 APA102, U7 APA102, U8 APA102

Commit message: Added gerbers, .gitignore and .gitattributes.
Parts:
- U1, U2, U3, U4, U5, U6, U7, U8: footprint Pete:APA102_2 -> Pete:APA102_3

Commit message: Fixes after double check.
Other:
- board text added: "1"
- board text added: "1/1"
- board text added: "2"
- board text added: "3"
- board text added: "4"
- board text added: "5"
- board text added: "5/19/17"
- board text added: "6"
- board text added: "7"
- board text added: "8"
- board text added: "HiBeam 8-pack"
- board text added: "Released under the Creative Commons Attribution Share-Alike 4.0 License https://creativecommons.org/licenses/by-sa/4.0/ Designed by Pete Dokter"
Changed lines of the file:
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@@
     (links 52)
     (no_connects 0)
-    (area 121.641205 72.114999 171.728795 120.952357)
+    (area 121.641205 72.114999 273.4474 194.4604)
     (thickness 1.6)
-    (drawings 16)
+    (drawings 40)
     (tracks 241)
     (zones 0)
@@
     (34 B.Paste user)
     (35 F.Paste user)
-    (36 B.SilkS user)
-    (37 F.SilkS user hide)
+    (36 B.SilkS user hide)
+    (37 F.SilkS user)
     (38 B.Mask user)
     (39 F.Mask user)
-    (40 Dwgs.User user hide)
+    (40 Dwgs.User user)
     (41 Cmts.User user)
     (42 Eco1.User user)
@@
     (pad_to_mask_clearance 0.2)
     (aux_axis_origin 0 0)
-    (visible_elements FFF9FF7F)
+    (visible_elements FFF8FF7F)
     (pcbplotparams
       (layerselection 0x000fc_ffffffff)
@@
     (pad 5 smd rect (at -2.399998 0 308.5) (size 2 1.1) (layers F.Cu F.Paste F.Mask)
       (net 16 "Net-(LED5-Pad5)") (solder_mask_margin 0.1016))
-    (pad 4 smd rect (at -2.4 -1.7 308.5) (size 2 1.1) (layers F.Cu F.Paste F.Mask)
+    (pad 4 smd rect (at -2.399999 -1.7 308.5) (size 2 1.1) (layers F.Cu F.Paste F.Mask)
       (net 1 +5V) (solder_mask_margin 0.1016))
     (pad 3 smd rect (at 2.4 -1.700001 128.5) (size 2 1.1) (layers F.Cu F.Paste F.Mask)
@@
     (pad 2 smd rect (at 2.399998 0 128.5) (size 2 1.1) (layers F.Cu F.Paste F.Mask)
       (net 13 "Net-(LED4-Pad5)") (solder_mask_margin 0.1016))
-    (pad 1 smd rect (at 2.4 1.7 128.5) (size 2 1.1) (layers F.Cu F.Paste F.Mask)
+    (pad 1 smd rect (at 2.399999 1.7 128.5) (size 2 1.1) (layers F.Cu F.Paste F.Mask)
       (net 14 "Net-(LED4-Pad6)") (solder_mask_margin 0.1016))
   )
@@
     (pad 5 smd rect (at -2.399998 0 102.8) (size 2 1.1) (layers F.Cu F.Paste F.Mask)
       (net 9 "Net-(LED2-Pad5)") (solder_mask_margin 0.1016))
-    (pad 4 smd rect (at -2.4 -1.7 102.8) (size 2 1.1) (layers F.Cu F.Paste F.Mask)
+    (pad 4 smd rect (at -2.4 -1.700001 102.8) (size 2 1.1) (layers F.Cu F.Paste F.Mask)
       (net 1 +5V) (solder_mask_margin 0.1016))
     (pad 3 smd rect (at 2.4 -1.700001 282.8) (size 2 1.1) (layers F.Cu F.Paste F.Mask)
@@
     (pad 2 smd rect (at 2.399998 0 282.8) (size 2 1.1) (layers F.Cu F.Paste F.Mask)
       (net 8 "Net-(LED1-Pad5)") (solder_mask_margin 0.1016))
-    (pad 1 smd rect (at 2.4 1.7 282.8) (size 2 1.1) (layers F.Cu F.Paste F.Mask)
+    (pad 1 smd rect (at 2.4 1.700001 282.8) (size 2 1.1) (layers F.Cu F.Paste F.Mask)
       (net 7 "Net-(LED1-Pad6)") (solder_mask_margin 0.1016))
   )
@@
     (fp_line (start -0.33782 0.4699) (end -0.33782 -0.48006) (layer Dwgs.User) (width 0.06604))
     (fp_line (start -0.8382 0.4699) (end -0.33782 0.4699) (layer Dwgs.User) (width 0.06604))
-    (pad 2 smd rect (at 0.84836 0 231.5) (size 1.09982 0.99822) (layers F.Cu F.Paste F.Mask)
+    (pad 2 smd rect (at 0.84836 0.000001 231.5) (size 1.09982 0.99822) (layers F.Cu F.Paste F.Mask)
       (net 2 GND))
-    (pad 1 smd rect (at -0.84836 0 231.5) (size 1.09982 0.99822) (layers F.Cu F.Paste F.Mask)
+    (pad 1 smd rect (at -0.84836 -0.000001 231.5) (size 1.09982 0.99822) (layers F.Cu F.Paste F.Mask)
       (net 1 +5V))
   )
@@
     (fp_line (start -0.33782 0.4699) (end -0.33782 -0.48006) (layer Dwgs.User) (width 0.06604))
     (fp_line (start -0.8382 0.4699) (end -0.33782 0.4699) (layer Dwgs.User) (width 0.06604))
-    (pad 2 smd rect (at 0.84836 0 128.5) (size 1.09982 0.99822) (layers F.Cu F.Paste F.Mask)
+    (pad 2 smd rect (at 0.84836 -0.000001 128.5) (size 1.09982 0.99822) (layers F.Cu F.Paste F.Mask)
       (net 2 GND))
-    (pad 1 smd rect (at -0.84836 0 128.5) (size 1.09982 0.99822) (layers F.Cu F.Paste F.Mask)
+    (pad 1 smd rect (at -0.84836 0.000001 128.5) (size 1.09982 0.99822) (layers F.Cu F.Paste F.Mask)
       (net 1 +5V))
   )
@@
       (net 2 GND))
   )
+  (gr_circle (center 145.542 110.744) (end 146.177 111.1758) (layer F.SilkS) (width 0.2))
+  (gr_circle (center 142.113 85.6234) (end 142.6972 86.106) (layer F.SilkS) (width 0.2))
+  (gr_circle (center 153.3144 86.614) (end 154.0256 86.8934) (layer F.SilkS) (width 0.2))
+  (gr_circle (center 156.083 106.7816) (end 156.7434 107.1626) (layer F.SilkS) (width 0.2))
+  (gr_circle (center 159.5882 96.0882) (end 160.274 96.393) (layer F.SilkS) (width 0.2))
+  (gr_circle (center 135.8138 104.9274) (end 136.3218 105.4862) (layer F.SilkS) (width 0.2))
+  (gr_circle (center 143.9926 94.2086) (end 144.6276 94.6404) (layer F.SilkS) (width 0.2))
+  (gr_circle (center 134.3152 93.726) (end 134.8994 94.2086) (layer F.SilkS) (width 0.2))
+  (gr_text 8 (at 145.5674 110.7186 154.3) (layer F.SilkS)
+    (effects (font (size 0.8128 0.8128) (thickness 0.1778)))
+  )
+  (gr_text 7 (at 156.0322 106.7054 205.7) (layer F.SilkS)
+    (effects (font (size 0.8128 0.8128) (thickness 0.1778)))
+  )
+  (gr_text 6 (at 159.5628 96.0882 257.2) (layer F.SilkS)
+    (effects (font (size 0.8128 0.8128) (thickness 0.1778)))
+  )
+  (gr_text 5 (at 153.2636 86.6394 308.5) (layer F.SilkS)
+    (effects (font (size 0.8128 0.8128) (thickness 0.1778)))
+  )
+  (gr_text 4 (at 142.0876 85.6488) (layer F.SilkS)
+    (effects (font (size 0.8128 0.8128) (thickness 0.1778)))
+  )
+  (gr_text 3 (at 134.3914 93.726 51.5) (layer F.SilkS)
+    (effects (font (size 0.8128 0.8128) (thickness 0.1778)))
+  )
+  (gr_text 2 (at 135.8392 104.902 102.8) (layer F.SilkS)
+    (effects (font (size 0.8128 0.8128) (thickness 0.1778)))
+  )
+  (gr_text 1 (at 143.9926 94.2086) (layer F.SilkS)
+    (effects (font (size 0.8128 0.8128) (thickness 0.1778)))
+  )
+  (dimension 8.8646 (width 0.3) (layer Dwgs.User)
+    (gr_text "0.3490 in" (at 126.8692 107.5563 90) (layer Dwgs.User)
+      (effects (font (size 1.5 1.2192) (thickness 0.3)))
+    )
+    (feature1 (pts (xy 146.685 103.124) (xy 125.5192 103.124)))
+    (feature2 (pts (xy 146.685 111.9886) (xy 125.5192 111.9886)))
+    (crossbar (pts (xy 128.2192 111.9886) (xy 128.2192 103.124)))
+    (arrow1a (pts (xy 128.2192 103.124) (xy 128.805621 104.250504)))
+    (arrow1b (pts (xy 128.2192 103.124) (xy 127.632779 104.250504)))
+    (arrow2a (pts (xy 128.2192 111.9886) (xy 128.805621 110.862096)))
+    (arrow2b (pts (xy 128.2192 111.9886) (xy 127.632779 110.862096)))
+  )
+  (dimension 14.1986 (width 0.3) (layer Dwgs.User)
+    (gr_text "0.5590 in" (at 153.7843 124.3876) (layer Dwgs.User)
+      (effects (font (size 1.5 1.5) (thickness 0.3)))
+    )
+    (feature1 (pts (xy 160.8836 103.124) (xy 160.8836 125.7376)))
+    (feature2 (pts (xy 146.685 103.124) (xy 146.685 125.7376)))
+    (crossbar (pts (xy 146.685 123.0376) (xy 160.8836 123.0376)))
+    (arrow1a (pts (xy 160.8836 123.0376) (xy 159.757096 123.624021)))
+    (arrow1b (pts (xy 160.8836 123.0376) (xy 159.757096 122.451179)))
+    (arrow2a (pts (xy 146.685 123.0376) (xy 147.811504 123.624021)))
+    (arrow2b (pts (xy 146.685 123.0376) (xy 147.811504 122.451179)))
+  )
+  (dimension 28.4226 (width 0.3) (layer Dwgs.User)
+    (gr_text "1.1190 in" (at 146.6977 129.5438) (layer Dwgs.User)
+      (effects (font (size 1.5 1.5) (thickness 0.3)))
+    )
+    (feature1 (pts (xy 132.4864 97.8916) (xy 132.4864 130.8938)))
+    (feature2 (pts (xy 160.909 97.8916) (xy 160.909 130.8938)))
+    (crossbar (pts (xy 160.909 128.1938) (xy 132.4864 128.1938)))
+    (arrow1a (pts (xy 132.4864 128.1938) (xy 133.612904 127.607379)))
+    (arrow1b (pts (xy 132.4864 128.1938) (xy 133.612904 128.780221)))
+    (arrow2a (pts (xy 160.909 128.1938) (xy 159.782496 127.607379)))
+    (arrow2b (pts (xy 160.909 128.1938) (xy 159.782496 128.780221)))
+  )
+  (gr_text 5/19/17 (at 212.3948 193.0146) (layer Dwgs.User)
+    (effects (font (size 1.5 1.5) (thickness 0.3)))
+  )
+  (gr_text v02 (at 271.2974 193.0654) (layer Dwgs.User)
+    (effects (font (size 1.5 1.5) (thickness 0.3)))
+  )
+  (gr_text 1/1 (at 188.468 183.1848) (layer Dwgs.User)
+    (effects (font (size 1.5 1.5) (thickness 0.3)))
+  )
+  (gr_text "HiBeam 8-pack" (at 195.9864 189.6618) (layer Dwgs.User)
+    (effects (font (size 1.5 1.5) (thickness 0.3)))
+  )
+  (gr_text "Released under the Creative Commons\nAttribution Share-Alike 4.0 License\nhttps://creativecommons.org/licenses/by-sa/4.0/\nDesigned by Pete Dokter" (at 178.435 173.5074) (layer Dwgs.User)
+    (effects (font (size 1.5 1.5) (thickness 0.3)) (justify left))
+  )
   (gr_text 5V (at 136.9822 101.854 22) (layer B.SilkS)

Commit message: Silk fixes.
Parts:
- moved ? 2.11 mm to (152.5, 91.9)
Other:
- rule pad_to_mask_clearance: 0.2 -> 0.1016
Changed lines of the file:
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@@
     (area 121.641205 72.114999 273.4474 194.4604)
     (thickness 1.6)
-    (drawings 40)
+    (drawings 39)
     (tracks 241)
     (zones 0)
@@
   (layers
     (0 F.Cu signal)
-    (31 B.Cu signal hide)
-    (32 B.Adhes user)
+    (31 B.Cu signal)
+    (32 B.Adhes user hide)
     (33 F.Adhes user hide)
-    (34 B.Paste user)
-    (35 F.Paste user)
-    (36 B.SilkS user hide)
+    (34 B.Paste user hide)
+    (35 F.Paste user hide)
+    (36 B.SilkS user)
     (37 F.SilkS user)
-    (38 B.Mask user)
+    (38 B.Mask user hide)
     (39 F.Mask user)
     (40 Dwgs.User user)
-    (41 Cmts.User user)
-    (42 Eco1.User user)
-    (43 Eco2.User user)
+    (41 Cmts.User user hide)
+    (42 Eco1.User user hide)
+    (43 Eco2.User user hide)
     (44 Edge.Cuts user)
-    (45 Margin user)
+    (45 Margin user hide)
     (46 B.CrtYd user hide)
     (47 F.CrtYd user hide)
-    (48 B.Fab user)
-    (49 F.Fab user)
+    (48 B.Fab user hide)
+    (49 F.Fab user hide)
   )
   (setup
@@
     (pad_size 1.524 1.524)
     (pad_drill 0.762)
-    (pad_to_mask_clearance 0.2)
+    (pad_to_mask_clearance 0.1016)
     (aux_axis_origin 0 0)
-    (visible_elements FFF8FF7F)
+    (visible_elements FFF9FF7F)
     (pcbplotparams
-      (layerselection 0x000fc_ffffffff)
+      (layerselection 0x010fc_ffffffff)
       (usegerberextensions false)
       (excludeedgelayer true)
@@
   )
   (module SparkFun:SFE_LOGO_NAME_FLAME_.1 (layer B.Cu)
-    (at 152.5524 93.98 180)
+    (at 152.5016 91.8718 180)
     (descr "SPARKFUN FONT LOGO W/ FLAME - 0.1\" HEIGHT - SILKSCREEN")
     (tags "SPARKFUN FONT LOGO W/ FLAME - 0.1\" HEIGHT - SILKSCREEN")
@@
       (net 2 GND))
   )
-  (gr_circle (center 145.542 110.744) (end 146.177 111.1758) (layer F.SilkS) (width 0.2))
-  (gr_circle (center 142.113 85.6234) (end 142.6972 86.106) (layer F.SilkS) (width 0.2))
-  (gr_circle (center 153.3144 86.614) (end 154.0256 86.8934) (layer F.SilkS) (width 0.2))
-  (gr_circle (center 156.083 106.7816) (end 156.7434 107.1626) (layer F.SilkS) (width 0.2))
-  (gr_circle (center 159.5882 96.0882) (end 160.274 96.393) (layer F.SilkS) (width 0.2))
-  (gr_circle (center 135.8138 104.9274) (end 136.3218 105.4862) (layer F.SilkS) (width 0.2))
-  (gr_circle (center 143.9926 94.2086) (end 144.6276 94.6404) (layer F.SilkS) (width 0.2))
-  (gr_circle (center 134.3152 93.726) (end 134.8994 94.2086) (layer F.SilkS) (width 0.2))
+  (gr_circle (center 145.542 110.744) (end 146.177 111.1758) (layer F.SilkS) (width 0.15))
+  (gr_circle (center 142.113 85.6234) (end 142.6972 86.106) (layer F.SilkS) (width 0.15))
+  (gr_circle (center 153.3144 86.614) (end 154.0256 86.8934) (layer F.SilkS) (width 0.15))
+  (gr_circle (center 156.083 106.7816) (end 156.7434 107.1626) (layer F.SilkS) (width 0.15))
+  (gr_circle (center 159.5882 96.0882) (end 160.274 96.393) (layer F.SilkS) (width 0.15))
+  (gr_circle (center 135.8138 104.9274) (end 136.3218 105.4862) (layer F.SilkS) (width 0.15))
+  (gr_circle (center 143.9926 94.2086) (end 144.6276 94.6404) (layer F.SilkS) (width 0.15))
+  (gr_circle (center 134.3152 93.726) (end 134.8994 94.2086) (layer F.SilkS) (width 0.15))
   (gr_text 8 (at 145.5674 110.7186 154.3) (layer F.SilkS)
     (effects (font (size 0.8128 0.8128) (thickness 0.1778)))
@@
     (effects (font (size 1.016 1.016) (thickness 0.2032)) (justify mirror))
   )
-  (gr_text "HiBeams 8-pack" (at 146.685 94.615) (layer B.SilkS)
-    (effects (font (size 1.016 1.016) (thickness 0.2032)) (justify mirror))
+  (gr_text "HiBeams 8-pack" (at 146.685 92.6592) (layer B.SilkS)
+    (effects (font (size 1.5 1.5) (thickness 0.3)) (justify mirror))
   )
   (gr_text v02 (at 159.7406 97.7646 90) (layer B.Cu)
@@
   (gr_circle (center 146.685 97.79) (end 157.226 107.315) (layer Edge.Cuts) (width 0.15))
   (gr_circle (center 146.685 97.79) (end 149.479 105.41) (layer Dwgs.User) (width 0.2))
-  (target plus (at 146.685 97.79) (size 5) (width 0.15) (layer Edge.Cuts))
   (segment (start 149.619135 106.301539) (end 149.6314 102.2858) (width 0.4064) (layer F.Cu) (net 1))
   (segment (start 149.6314 102.2858) (end 150.508101 101.851562) (width 0.4064) (layer F.Cu) (net 1))
